Commit message: Controlador de posicion del padlet

File: description/ros2_control.xacro (robot description, xacro)
@@ -66,12 +66,12 @@
                 <state_interface name="position"/>
             </joint>
-            <!-- <joint name="padlet_joint">
+            <joint name="padlet_joint">
                 <command_interface name="position">
-                    <param name="min">-0.785</param>
-                    <param name="max">0.785</param>
+                    <param name="min">-1</param>
+                    <param name="max">1</param>
                 </command_interface>
+                <!-- <state_interface name="position"/> -->
                 <state_interface name="position"/>
-                <state_interface name="velocity"/>
-            </joint> -->
+            </joint>
         </ros2_control>
     </xacro:if>
