Commit message: Padlet carga en Gazebo C:

File: description/padlet.xacro (robot description, xacro)
@@ -20,6 +20,6 @@
             </geometry>
         </collision>
-        <xacro:inertial_box mass="0.5" x="0.5" y="0.25" z="0.15">
-            <origin xyz="0 0 0.075" rpy="0 0 0"/>
+        <xacro:inertial_box mass="2" x="0.5" y="0.25" z="0.15">
+            <origin xyz="0 0 0.0" rpy="0 0 0"/>
         </xacro:inertial_box>
     </link>
@@ -32,5 +32,5 @@
     </joint>
     <gazebo reference="base_padlet">
-        <material>Gazebo/Green</material>
+        <material>Gazebo/Grey</material>
     </gazebo>
 </robot>

File: description/robot.urdf.xacro (robot description, xacro)
@@ -13,5 +13,5 @@
     <xacro:include filename="camera.xacro" />
     <!-- <xacro:include filename="depth_camera.xacro" /> -->
-    <!-- <xacro:include filename= 'padlet.xacro'/>-->
+    <xacro:include filename= 'padlet.xacro'/>
     <xacro:include filename="face.xacro" />
 </robot>

File: description/robot_core.xacro (robot description, xacro)
@@ -62,10 +62,10 @@
             </geometry>
         </collision>
-        <xacro:inertial_box mass="0.5" x="${chassis_length}" y="${chassis_width}" z="${chassis_height}">
+        <xacro:inertial_box mass="5" x="${chassis_length}" y="${chassis_width}" z="${chassis_height}">
             <origin xyz="${chassis_length/2} 0 ${chassis_height/2}" rpy="0 0 0"/>
         </xacro:inertial_box>
     </link>
     <gazebo reference="chassis">
-        <material>Gazebo/Green</material>
+        <material>Gazebo/Red</material>
     </gazebo>
     <!-- LEFT WHEEL LINK -->

Commit message: posibles arreglos de controlador

File: description/padlet.xacro (robot description, xacro)
@@ -32,5 +32,19 @@
     </joint>
     <gazebo reference="base_padlet">
-        <material>Gazebo/Grey</material>
+        <material>Gazebo/White</material>
     </gazebo>
+    <!-- <gazebo>
+        <plugin name="gazebo_ros_joint_state_publisher"
+            filename="libgazebo_ros_joint_state_pubisher">
+            <update_rate>20</update_rate>
+            <joint_name>padlet_joint</joint_name>
+        </plugin>
+    </gazebo>
+    <gazebo>
+        <plugin name="gazebo_ros_joint_pose_trajectory"
+            filename="libgazebo_ros_joint_pose_trajectory.so">
+            <update_rate>20</update_rate>
+        </plugin>
+    </gazebo>
+     -->
 </robot>

File: description/ros2_control.xacro (robot description, xacro)
@@ -30,4 +30,18 @@
             </joint>
         </ros2_control>
+        <!-- <ros2_control name="GazeboSimSystem" type="system">
+            <hardware>
+                <plugin>gz_ros2_control/GazeboSimSystem</plugin>
+            </hardware>
+            <joint name="padlet_joint">
+                <command_interface name="position">
+                    <param name="min">-0.785</param>
+                    <param name="max">0.785</param>
+                </command_interface>
+                <state_interface name="position">
+                    <param name="initial_value">1.0</param>
+                </state_interface>
+            </joint>
+        </ros2_control> -->
     </xacro:unless>
     <xacro:if value="$(arg sim_mode)">
@@ -52,4 +66,12 @@
                 <state_interface name="position"/>
             </joint>
+            <!-- <joint name="padlet_joint">
+                <command_interface name="position">
+                    <param name="min">-0.785</param>
+                    <param name="max">0.785</param>
+                </command_interface>
+                <state_interface name="position"/>
+                <state_interface name="velocity"/>
+            </joint> -->
         </ros2_control>
     </xacro:if>

Commit message: control de trayectoria

File: description/padlet.xacro (robot description, xacro)
@@ -24,5 +24,5 @@
         </xacro:inertial_box>
     </link>
-    <joint name="padlet_joint" type="revolute">
+    <joint name="padlet_joint" type="continuous">
         <parent link="chassis"/>
         <child link="base_padlet"/>

File: description/ros2_control.xacro (robot description, xacro)
@@ -71,5 +71,9 @@
                     <param name="max">1</param>
                 </command_interface>
-                <!-- <state_interface name="position"/> -->
+                <!-- <command_interface name="velocity">
+                    <param name="min">-3</param>
+                    <param name="max">10</param>
+                </command_interface> -->
+                <state_interface name="velocity"/>
                 <state_interface name="position"/>
             </joint>
